File: PCB/FlightBridgePCB/FlightBridgePCB.kicad_pcb (KiCad board)
At the start: 2 copper layers, 65 x 35 mm, 12 parts, among them J1 Raspberry_Pi_2_3, J2 AVR-ISP-6, U1 ATmega128A-AU, Y1 Crystal

Commit message: PCB Update
Parts:
- removed the REF** at (161.5, 46.5)
- removed the REF** at (161.5, 18.5)
- removed the REF** at (103.5, 46.5)
- removed the REF** at (103.5, 18.5)
- added REF**: MountingHole_2.7mm_M2.5, MountingHole:MountingHole_2.7mm_M2.5, F.Cu at (171.7, 94.5)
- added REF**: MountingHole_2.7mm_M2.5, MountingHole:MountingHole_2.7mm_M2.5, F.Cu at (171.7, 71.5)
- added REF**: MountingHole_2.7mm_M2.5, MountingHole:MountingHole_2.7mm_M2.5, F.Cu at (113.7, 94.5)
- added REF**: MountingHole_2.7mm_M2.5, MountingHole:MountingHole_2.7mm_M2.5, F.Cu at (113.7, 71.5)
- J2: footprint Connector_PinSocket_2.54mm:PinSocket_2x03_P2.54mm_Vertical -> Connector_PinHeader_2.54mm:PinHeader_2x03_P2.54mm_Vertical
- moved C2 76.1 mm to (160.3, 94.9)
- moved Y1 71.3 mm to (161.4, 86.2), turned to 270 degrees
- moved C1 58.2 mm to (160.3, 77.1), turned to 180 degrees
- moved J2 56.2 mm to (170.5, 81.0)
- moved ? 54.0 mm to (126.7, 81.3)
- moved J1 54.0 mm to (118.6, 72.8)
- moved R1 54.0 mm to (131.8, 85.5)
- moved U1 52.6 mm to (146.0, 86.3), turned to 135 degrees
Other:
- board size 65 x 35 mm -> 65 x 30 mm

Commit message: First Full PCB
Parts:
- added D1: LED, LED_SMD:LED_0805_2012Metric_Castellated, F.Cu at (141.0, 94.5)
- added D2: LED, LED_SMD:LED_0805_2012Metric_Castellated, F.Cu at (144.0, 94.5)
- added D3: LED, LED_SMD:LED_0805_2012Metric_Castellated, F.Cu at (147.5, 94.5)
- added D4: LED, LED_SMD:LED_0805_2012Metric_Castellated, F.Cu at (123.9, 76.4)
- added D5: LED, LED_SMD:LED_0805_2012Metric_Castellated, F.Cu at (124.0, 79.8)
- added J3: Conn_01x05, Connector_PinHeader_2.54mm:PinHeader_1x05_P2.54mm_Horizontal, F.Cu at (114.0, 88.5)
- added J4: Conn_01x03, Connector_PinHeader_2.54mm:PinHeader_1x03_P2.54mm_Horizontal, F.Cu at (125.0, 94.0)
- added J5: Conn_01x04, Connector_PinHeader_2.54mm:PinHeader_1x04_P2.54mm_Horizontal, F.Cu at (137.0, 94.0)
- added R2: 300, Resistor_SMD:R_0805_2012Metric_Pad1.20x1.40mm_HandSolder, F.Cu at (141.0, 90.0)
- added R3: 300, Resistor_SMD:R_0805_2012Metric_Pad1.20x1.40mm_HandSolder, F.Cu at (144.0, 90.0)
- added R4: 300, Resistor_SMD:R_0805_2012Metric_Pad1.20x1.40mm_HandSolder, F.Cu at (147.5, 90.0)
- added R5: 300, Resistor_SMD:R_0805_2012Metric_Pad1.20x1.40mm_HandSolder, F.Cu at (119.7, 76.4)
- added R6: 300, Resistor_SMD:R_0805_2012Metric_Pad1.20x1.40mm_HandSolder, F.Cu at (119.7, 79.8)
- added R7: 0, Resistor_SMD:R_0805_2012Metric_Pad1.20x1.40mm_HandSolder, F.Cu at (119.0, 87.0)
- added R8: 0, Resistor_SMD:R_0805_2012Metric_Pad1.20x1.40mm_HandSolder, F.Cu at (119.0, 89.5)
- moved R1 40.6 mm to (171.8, 78.2)
- moved C2 19.3 mm to (167.5, 77.0), turned to 180 degrees
- moved U1 12.7 mm to (158.5, 88.5), turned to 180 degrees
- moved C1 11.4 mm to (149.0, 77.0)
- moved Y1 9.73 mm to (158.2, 77.0), turned to 0 degrees
- moved ? 7.00 mm to (133.7, 81.3)
- moved J2 5.70 mm to (172.8, 86.2), turned to 180 degrees
Connections:
- J1 pad 10: Net-(J1-Pad10) -> UART_TELEM_PI
- J1 pad 15: Net-(J1-Pad15) -> ABORT
- J1 pad 16: Net-(J1-Pad16) -> SUPERVISOR_RESET
- J1 pad 8: Net-(J1-Pad8) -> UART_SBUS
- U1 pad 2: Net-(U1-Pad2) -> UART_SBUS
- U1 pad 27: Net-(U1-Pad27) -> UART_TELEM
- U1 pad 28: Net-(U1-Pad28) -> UART_RESET
- U1 pad 3: Net-(U1-Pad3) -> UART_TELEM_PI
- U1 pad 35: Net-(U1-Pad35) -> ABORT
- U1 pad 36: Net-(U1-Pad36) -> SUPERVISOR_RESET
- U1 pad 45: Net-(U1-Pad45) -> AUX2
- U1 pad 46: Net-(U1-Pad46) -> AUX1
- U1 pad 47: Net-(U1-Pad47) -> N
- U1 pad 48: Net-(U1-Pad48) -> R
- U1 pad 49: Net-(U1-Pad49) -> A
Routing:
- net +3V3: track 0.00 -> 121.2 mm, vias 0 -> 16
- net UART_SBUS: track 0.00 -> 81.8 mm, vias 0 -> 2
- net UART_TELEM_PI: track 0.00 -> 54.4 mm, vias 0 -> 2
- net UART_RESET: track 0.00 -> 47.7 mm, vias 0 -> 2
- net GND: track 0.00 -> 44.4 mm, vias 0 -> 4
- net UART_TELEM: track 0.00 -> 44.3 mm, vias 0 -> 2
- net +5V: track 0.00 -> 40.6 mm, vias 0 -> 3
- net AUX2: track 0.00 -> 29.2 mm, vias 0 -> 2
- net SUPERVISOR_RESET: track 0.00 -> 27.2 mm
- net AUX1: track 0.00 -> 27.1 mm, vias 0 -> 2
- net A: track 0.00 -> 24.7 mm, vias 0 -> 2
- net ABORT: track 0.00 -> 21.7 mm
- net R: track 0.00 -> 18.5 mm, vias 0 -> 2
- net ~RST~: track 0.00 -> 14.6 mm
- net MISO: track 0.00 -> 13.4 mm
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- added copper zone on B.Cu, net GND

Commit message: PCB Updates
Parts:
- added G***: LOGO, FlightBridgePCB:Astro, F.Cu at (132.3, 81.0)
Routing:
- net +5V: track 40.6 -> 41.8 mm
- net +3V3: vias 16 -> 15
Other:
- board text added: "3V3"
- board text added: "5V"
- board text added: "AUX1"
- board text added: "AUX2"
- board text added: "CLI"
- board text added: "EXT Telem"
- board text added: "FC CLI (RESET)"
- board text added: "FC Telem"
- board text added: "FlightBridge Rev 1 Connor Raggatt 04/2021"
- board text added: "GND"
- board text added: "MOSI"
- board text added: "Pi Telem"
- board text added: "SBUS"

Commit message: First PCB to be Built
Parts:
- added C3: 1uf, Capacitor_SMD:C_0805_2012Metric_Pad1.18x1.45mm_HandSolder, F.Cu at (127.3, 77.1)
- added C4: 1uf, Capacitor_SMD:C_0805_2012Metric_Pad1.18x1.45mm_HandSolder, F.Cu at (135.1, 77.1)
- added C5: 1u, Capacitor_SMD:C_0805_2012Metric_Pad1.18x1.45mm_HandSolder, B.Cu at (122.8, 78.9)
- added C6: 1u, Capacitor_SMD:C_0805_2012Metric_Pad1.18x1.45mm_HandSolder, B.Cu at (122.7, 80.9)
- added C7: 1u, Capacitor_SMD:C_0805_2012Metric_Pad1.18x1.45mm_HandSolder, F.Cu at (168.0, 78.0)
- added C8: 1u, Capacitor_SMD:C_0805_2012Metric_Pad1.18x1.45mm_HandSolder, F.Cu at (170.4, 89.4)
- added Q1: IRF3205, Package_TO_SOT_THT:TO-220-3_Vertical, F.Cu at (120.0, 88.9)
- added Q2: BC849, Package_TO_SOT_SMD:SOT-23, F.Cu at (124.6, 88.5)
- added R10: 1k, Resistor_SMD:R_0805_2012Metric_Pad1.20x1.40mm_HandSolder, F.Cu at (128.9, 89.4)
- added R9: 100k, Resistor_SMD:R_0805_2012Metric_Pad1.20x1.40mm_HandSolder, F.Cu at (123.8, 84.4)
- added U2: L78L33_TO92, Package_TO_SOT_THT:TO-92_Inline, F.Cu at (132.5, 77.3)
- J3: value Conn_01x05 -> Conn_01x04; footprint Connector_PinHeader_2.54mm:PinHeader_1x05_P2.54mm_Horizontal -> Connector_PinHeader_2.54mm:PinHeader_1x04_P2.54mm_Horizontal
- J4: footprint Connector_PinHeader_2.54mm:PinHeader_1x03_P2.54mm_Horizontal -> FlightBridgePCB:EXTERNAL_TELEM
- J5: value Conn_01x04 -> Conn_01x03; footprint Connector_PinHeader_2.54mm:PinHeader_1x04_P2.54mm_Horizontal -> FlightBridgePCB:ELECTRICAL_Connection
- moved J5 26.8 mm to (112.5, 83.1), turned to 90 degrees
- moved J3 24.0 mm to (137.4, 93.9), turned to 270 degrees
- moved R7 16.6 mm to (135.3, 90.2)
- moved G*** 11.2 mm to (143.4, 82.7)
- moved D5 6.78 mm to (118.6, 75.7), turned to 0 degrees
- moved R8 5.75 mm to (123.7, 92.8), turned to 270 degrees
- moved D4 5.66 mm to (118.7, 78.5), turned to 0 degrees
- moved R6 5.08 mm to (122.7, 75.7), turned to 180 degrees
- moved J4 4.06 mm to (121.0, 94.9), turned to 0 degrees
- moved R5 3.65 mm to (122.7, 78.5), turned to 180 degrees
- moved C1 2.14 mm to (150.9, 76.1), turned to 90 degrees
- moved C2 1.40 mm to (168.0, 75.7)
- moved Y1 0.89 mm to (159.1, 77.0)
- moved R1 0.44 mm to (172.1, 78.0)
- moved D2 0.25 mm to (144.3, 94.5)
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Connections:
- J1 pad 1: +3V3 -> Net-(J1-Pad1)
- J1 pad 14: GND -> GND1
- J1 pad 17: +3V3 -> Net-(J1-Pad17)
- J1 pad 20: GND -> GND1
- J1 pad 25: GND -> GND1
- J1 pad 30: GND -> GND1
- J1 pad 34: GND -> GND1
- J1 pad 39: GND -> GND1
- J1 pad 6: GND -> GND1
- J1 pad 9: GND -> GND1
- J3 pad 2: GND -> GND1
- J5 pad 1: +3V3 -> GND1
- J5 pad 3: AUX1 -> Vin
- U1 pad 28: UART_RESET -> Net-(U1-Pad28)
- U1 pad 45: AUX2 -> Net-(U1-Pad45)
- U1 pad 46: AUX1 -> ~POWER_EN~
Routing:
- net GND1: track 0.00 -> 103.9 mm, vias 0 -> 9
- net UART_RESET: track 47.7 -> 0.00 mm, vias 2 -> 0
- net AUX2: track 29.2 -> 0.00 mm, vias 2 -> 0
- net Vin: track 0.00 -> 28.2 mm, vias 0 -> 1
- net AUX1: track 27.1 -> 0.00 mm, vias 2 -> 0
- net ~POWER_EN~: track 0.00 -> 23.3 mm, vias 0 -> 2
- net +5V: track 41.8 -> 63.3 mm, vias 3 -> 4
- net +3V3: track 121.2 -> 107.6 mm, vias 15 -> 6
- net UART_SBUS: track 81.8 -> 68.4 mm, vias 2 -> 5
- net Net-(Q1-Pad1): track 0.00 -> 6.91 mm
- net GND: track 44.4 -> 51.0 mm, vias 4 -> 15
- net N: track 7.59 -> 10.8 mm, vias 0 -> 2
- net UART_TELEM_EXT: track 5.30 -> 2.37 mm
- net Net-(Q2-Pad1): track 0.00 -> 2.36 mm
- net ABORT: track 21.7 -> 24.1 mm
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- added copper zone on F.Cu, net GND
- added copper zone on B.Cu, net GND1
- added copper zone on F.Cu, net GND1
Other:
- board text added: "A"
- board text added: "ExTelem"
- board text added: "FC TELEM"
- board text added: "FlightBridge Rev 2 Connor Raggatt 18/04/2021"
- board text added: "GND1 (Switched)"
- board text added: "JLCJLCJLCJLC"
- board text added: "N"
- board text added: "R"
- board text added: "TELEM PI"
- board text added: "VBAT"
- board text removed: "AUX1"
- board text removed: "AUX2"
- board text removed: "CLI"
- board text removed: "EXT Telem"
- board text removed: "FC CLI (RESET)"
- board text removed: "FlightBridge Rev 1 Connor Raggatt 04/2021"
- board text removed: "Pi Telem"

Commit message: New PCB
Parts:
- removed ?: , 
- removed R7, R8: 0, Resistor_SMD:R_0805_2012Metric_Pad1.20x1.40mm_HandSolder
- J3: value Conn_01x04 -> Conn_01x03; footprint Connector_PinHeader_2.54mm:PinHeader_1x04_P2.54mm_Horizontal -> Connector_PinHeader_2.54mm:PinHeader_1x03_P2.54mm_Horizontal
- J4: value Conn_01x03 -> Conn_01x04; footprint FlightBridgePCB:EXTERNAL_TELEM -> Connector_PinHeader_2.54mm:PinHeader_1x04_P2.54mm_Horizontal
- U2: value L78L33_TO92 -> MCP1700-3302E_TO92
- moved J4 7.83 mm to (128.8, 93.7), turned to 270 degrees
- moved U2 2.42 mm to (130.0, 77.5), turned to 0 degrees
- moved G*** 0.18 mm to (143.3, 82.5)
- moved J3 0.13 mm to (137.4, 93.7)
Connections:
- J1 pad 3: Net-(J1-Pad3) -> SDA
- J1 pad 5: Net-(J1-Pad5) -> SCL
- J1 pad 8: UART_SBUS -> MOSI
- J3 pad 3: UART_TELEM_FC -> MOSI
- J4 pad 1: +5V -> +3V3
- J4 pad 3: UART_TELEM_EXT -> SDA
- U1 pad 12: MOSI -> Net-(U1-Pad12)
- U1 pad 13: MISO -> Net-(U1-Pad13)
- U1 pad 2: UART_SBUS -> MOSI
- U1 pad 27: UART_TELEM -> Net-(U1-Pad27)
- U1 pad 3: UART_TELEM_PI -> MISO
- U2 pad 1: +3V3 -> GND
- U2 pad 2: GND -> Vin
- U2 pad 3: Vin -> +3V3
Routing:
- net MOSI: track 4.83 -> 83.2 mm, vias 0 -> 6
- net UART_SBUS: track 68.4 -> 0.00 mm, vias 5 -> 0
- net SCL: track 0.00 -> 53.1 mm, vias 0 -> 5
- net UART_TELEM_PI: track 52.9 -> 0.00 mm, vias 2 -> 0
- net SDA: track 0.00 -> 50.9 mm, vias 0 -> 5
- net UART_TELEM: track 43.8 -> 0.00 mm, vias 4 -> 0
- net +3V3: track 107.6 -> 125.1 mm, vias 6 -> 8
- net GND: track 51.0 -> 41.8 mm, vias 15 -> 14
- net +5V: track 63.3 -> 70.6 mm
- net GND1: track 103.9 -> 97.0 mm
- net UART_TELEM_FC: track 5.10 -> 0.00 mm
- net Vin: track 28.2 -> 30.8 mm
- net UART_TELEM_EXT: track 2.37 -> 0.00 mm
- net MISO: track 12.8 -> 11.5 mm, vias 0 -> 1
Other:
- board text added: "FlightBridge Rev 3 Connor Raggatt 6/05/2021"
- board text removed: "ExTelem"
- board text removed: "FlightBridge Rev 2 Connor Raggatt 18/04/2021"
