File: PCB/FlightBridgePCB/FlightBridgePCB.sch (KiCad schematic (older format))
At the start: 7 parts, among them J1 Raspberry_Pi_2_3, J2 AVR-ISP-6, U1 ATmega128A-AU, Y1 Crystal

Commit message: PCB Update
Parts:
- added J?: Conn_01x05, symbol Connector_Generic:Conn_01x05
- added J?: Conn_01x03, symbol Connector_Generic:Conn_01x03
- added R? (x2): 0, symbol Device:R
- J2: footprint Connector_PinSocket_2.54mm:PinSocket_2x03_P2.54mm_Vertical -> Connector_PinHeader_2.54mm:PinHeader_2x03_P2.54mm_Vertical
Connections:
- net +5V: now also J?.1 (Pin_1), J?.1 (Pin_1)
- net GND: now also J?.2 (Pin_2), J?.2 (Pin_2)
- net UART_SBUS: now reaches U1.2 (PE0)
- net UART_SBUS: now also J1.8 (GPIO14/TXD), J?.3 (Pin_3)
- net UART_RESET: now reaches U1.28 (PD3)
- net UART_RESET: now also J?.5 (Pin_5)
- net UART_TELEM: now reaches J1.10 (GPIO15/RXD)
- net UART_TELEM: now also R?.1, R?.2
- new net UART_TELEM_EXT: J?.3 (Pin_3), R?.2
- new net UART_TELEM_FC: J?.4 (Pin_4), R?.1
Other:
- note added: "ATmega ISP Header\n"
- note added: "External Telemetry"
- note added: "Telemetry Selector\n"
Changed lines of the file:
@@
 encoding utf-8
 Sheet 1 1
-Title ""
-Date ""
-Rev ""
-Comp ""
-Comment1 ""
+Title "FlightBridge PCB"
+Date "2021-03-30"
+Rev "1"
+Comp "METR4810 Team 8"
+Comment1 "Connor Raggatt"
 Comment2 ""
 Comment3 ""
@@
 F 0 "J2" H 3721 6296 50  0000 R CNN
 F 1 "AVR-ISP-6" H 3721 6205 50  0000 R CNN
-F 2 "Connector_PinSocket_2.54mm:PinSocket_2x03_P2.54mm_Vertical" V 3800 6250 50  0001 C CNN
+F 2 "Connector_PinHeader_2.54mm:PinHeader_2x03_P2.54mm_Vertical" V 3800 6250 50  0001 C CNN
 F 3 " ~" H 2775 5650 50  0001 C CNN
 	1    4050 6200
@@
 	1    0    0    -1
 $EndComp
+$Comp
+L Connector_Generic:Conn_01x05 J?
+U 1 1 606579CB
+P 9700 2200
+F 0 "J?" H 9780 2242 50  0000 L CNN
+F 1 "Conn_01x05" H 9780 2151 50  0000 L CNN
+F 2 "" H 9700 2200 50  0001 C CNN
+F 3 "~" H 9700 2200 50  0001 C CNN
+	1    9700 2200
+	1    0    0    -1
+$EndComp
+$Comp
+L power:+5V #PWR?
+U 1 1 60658AB4
+P 9500 2000
+F 0 "#PWR?" H 9500 1850 50  0001 C CNN
+F 1 "+5V" V 9515 2128 50  0000 L CNN
+F 2 "" H 9500 2000 50  0001 C CNN
+F 3 "" H 9500 2000 50  0001 C CNN
+	1    9500 2000
+	0    -1   -1   0
+$EndComp
+$Comp
+L power:GND #PWR?
+U 1 1 60659B5F
+P 9500 2100
+F 0 "#PWR?" H 9500 1850 50  0001 C CNN
+F 1 "GND" V 9505 1972 50  0000 R CNN
+F 2 "" H 9500 2100 50  0001 C CNN
+F 3 "" H 9500 2100 50  0001 C CNN
+	1    9500 2100
+	0    1    1    0
+$EndComp
+Text GLabel 1350 2500 0    50   Output ~ 0
+UART_SBUS
+Text GLabel 1350 2600 0    50   Input ~ 0
+UART_TELEM
+Text GLabel 5300 4800 0    50   Input ~ 0
+UART_SBUS
+Text GLabel 9500 2200 0    50   Input ~ 0
+UART_SBUS
+Text GLabel 9500 2300 0    50   Output ~ 0
+UART_TELEM_FC
+Text Notes 3650 5400 0    50   ~ 0
+ATmega ISP Header\n
+Text GLabel 6500 5100 2    50   Output ~ 0
+UART_RESET
+Text GLabel 9500 2400 0    50   Input ~ 0
+UART_RESET
+$Comp
+L Device:R R?
+U 1 1 606721A0
+P 9700 3250
+F 0 "R?" H 9770 3296 50  0000 L CNN
+F 1 "0" H 9770 3205 50  0000 L CNN
+F 2 "" V 9630 3250 50  0001 C CNN
+F 3 "~" H 9700 3250 50  0001 C CNN
+	1    9700 3250
+	1    0    0    -1
+$EndComp
+$Comp
+L Device:R R?
+U 1 1 60672D84
+P 9700 3550
+F 0 "R?" H 9770 3596 50  0000 L CNN
+F 1 "0" H 9770 3505 50  0000 L CNN
+F 2 "" V 9630 3550 50  0001 C CNN
+F 3 "~" H 9700 3550 50  0001 C CNN
+	1    9700 3550
+	1    0    0    -1
+$EndComp
+Text GLabel 9550 3400 0    50   Output ~ 0
+UART_TELEM
+Wire Wire Line
+	9550 3400 9700 3400
+Connection ~ 9700 3400
+Text Notes 9150 2900 0    50   ~ 0
+Telemetry Selector\n
+Text GLabel 10000 3100 2    50   Input ~ 0
+UART_TELEM_FC
+Wire Wire Line
+	9700 3100 10000 3100
+$Comp
+L Connector_Generic:Conn_01x03 J?
+U 1 1 6067E30D
+P 9700 4800
+F 0 "J?" H 9780 4842 50  0000 L CNN
+F 1 "Conn_01x03" H 9780 4751 50  0000 L CNN
+F 2 "" H 9700 4800 50  0001 C CNN
+F 3 "~" H 9700 4800 50  0001 C CNN
+	1    9700 4800
+	1    0    0    -1
+$EndComp
+Text Notes 9350 4400 0    50   ~ 0
+External Telemetry
+Text GLabel 9500 4900 0    50   Output ~ 0
+UART_TELEM_EXT
+$Comp
+L power:+5V #PWR?
+U 1 1 6068215D
+P 9500 4700
+F 0 "#PWR?" H 9500 4550 50  0001 C CNN
+F 1 "+5V" V 9515 4828 50  0000 L CNN
+F 2 "" H 9500 4700 50  0001 C CNN
+F 3 "" H 9500 4700 50  0001 C CNN
+	1    9500 4700
+	0    -1   -1   0
+$EndComp
+$Comp
+L power:GND #PWR?
+U 1 1 60682A5F
+P 9500 4800
+F 0 "#PWR?" H 9500 4550 50  0001 C CNN
+F 1 "GND" V 9505 4672 50  0000 R CNN
+F 2 "" H 9500 4800 50  0001 C CNN
+F 3 "" H 9500 4800 50  0001 C CNN
+	1    9500 4800
+	0    1    1    0
+$EndComp
+Text GLabel 10000 3700 2    50   Input ~ 0
+UART_TELEM_EXT
+Wire Wire Line
+	9700 3700 10000 3700
 $EndSCHEMATC

Commit message: First Full PCB
Parts:
- added D1, D2, D3, D4, D5: LED, LED_SMD:LED_0805_2012Metric_Castellated, symbol Device:LED
- added J5: Conn_01x04, Connector_PinHeader_2.54mm:PinHeader_1x04_P2.54mm_Horizontal, symbol Connector_Generic:Conn_01x04
- added R2, R3, R4, R5, R6: 300, Resistor_SMD:R_0805_2012Metric_Pad1.20x1.40mm_HandSolder, symbol Device:R
- J3: renamed from J?; footprint (none) -> Connector_PinHeader_2.54mm:PinHeader_1x05_P2.54mm_Horizontal
- J4: renamed from J?; footprint (none) -> Connector_PinHeader_2.54mm:PinHeader_1x03_P2.54mm_Horizontal
- R7, R8: renamed from R?; footprint (none) -> Resistor_SMD:R_0805_2012Metric_Pad1.20x1.40mm_HandSolder
Connections:
- net +3V3: now also J5.1 (Pin_1), R5.1
- net +5V: now also R6.1
- net GND: now also D1.1 (K), D2.1 (K), D3.1 (K), D4.1 (K), D5.1 (K), J5.2 (Pin_2)
- net UART_SBUS: now also J3.4 (Pin_4); no longer J3.3 (Pin_3)
- net UART_TELEM: now also U1.27 (PD2); no longer J1.10 (GPIO15/RXD)
- net UART_TELEM_FC: now also J3.3 (Pin_3); no longer J3.4 (Pin_4)
- net UART_TELEM_PI: now reaches U1.3 (PE1)
- net UART_TELEM_PI: now also J1.10 (GPIO15/RXD)
- net ABORT: now reaches U1.35 (PC0)
- net ABORT: now also J1.15 (GPIO22)
- net SUPERVISOR_RESET: now reaches U1.36 (PC1)
- net SUPERVISOR_RESET: now also J1.16 (GPIO23)
- net AUX2: now reaches U1.45 (PA6)
- net AUX2: now also J5.4 (Pin_4)
- net AUX1: now reaches U1.46 (PA5)
- net AUX1: now also J5.3 (Pin_3)
- net N: now reaches U1.47 (PA4)
- net N: now also R4.1
- net R: now reaches U1.48 (PA3)
- net R: now also R3.1
- net A: now reaches U1.49 (PA2)
- net A: now also R2.1
- new net: D3.2 (A), R4.2
- new net: D4.2 (A), R5.2
- new net: D5.2 (A), R6.2
- new net: D2.2 (A), R3.2
- new net: D1.2 (A), R2.2
Other:
- note added: "Additional GPIO Output for Power Switching (if necessary)\n"
- note added: "External Telemetry Input\n"
- note added: "Indicator LEDs\n"
- note removed: "External Telemetry"
- moved on the sheet: J3, J4, R7, R8

Commit message: First PCB to be Built
Parts:
- removed J3: Conn_01x05, Connector_PinHeader_2.54mm:PinHeader_1x05_P2.54mm_Horizontal, symbol Connector_Generic:Conn_01x05
- removed J5: Conn_01x04, Connector_PinHeader_2.54mm:PinHeader_1x04_P2.54mm_Horizontal, symbol Connector_Generic:Conn_01x04
- added C3, C4: 1uf, Capacitor_SMD:C_0805_2012Metric_Pad1.18x1.45mm_HandSolder, symbol Device:C
- added C5, C6, C7, C8: 1u, Capacitor_SMD:C_0805_2012Metric_Pad1.18x1.45mm_HandSolder, symbol Device:C
- added J3: Conn_01x04, Connector_PinHeader_2.54mm:PinHeader_1x04_P2.54mm_Horizontal, symbol Connector_Generic:Conn_01x04
- added J5: Conn_01x03, FlightBridgePCB:ELECTRICAL_Connection, symbol Connector_Generic:Conn_01x03
- added Q1: IRF3205, Package_TO_SOT_THT:TO-220-3_Vertical, symbol Transistor_FET:IRF3205
- added Q2: BC849, Package_TO_SOT_SMD:SOT-23, symbol Transistor_BJT:BC849
- added R10: 1k, Resistor_SMD:R_0805_2012Metric_Pad1.20x1.40mm_HandSolder, symbol Device:R
- added R9: 100k, Resistor_SMD:R_0805_2012Metric_Pad1.20x1.40mm_HandSolder, symbol Device:R
- added U2: L78L33_TO92, Package_TO_SOT_THT:TO-92_Inline, symbol Regulator_Linear:L78L33_TO92
- J4: footprint Connector_PinHeader_2.54mm:PinHeader_1x03_P2.54mm_Horizontal -> FlightBridgePCB:EXTERNAL_TELEM
Connections:
- net +3V3: now also C4.1, C7.1, C8.1, U2.1 (VO); no longer J1.1 (3V3), J1.17 (3V3)
- net +5V: now also C5.1, C6.1, J3.1 (Pin_1)
- net GND: now also C3.2, C4.2, C5.2, C6.2, C7.2, C8.2, J5.2 (Pin_2), Q1.3 (S), Q2.2 (E), U2.2 (GND); no longer J1.14 (GND), J1.20 (GND), J1.25 (GND), J1.30 (GND), J1.34 (GND), J1.39 (GND), J1.6 (GND), J1.9 (GND)
- net UART_SBUS: now also J3.4 (Pin_4)
- net UART_TELEM_FC: now also J3.3 (Pin_3)
- net AUX1 renamed ~POWER_EN~
- net ~POWER_EN~: now also R10.2
- net AUX2: no longer names the net of U1.45 (PA6)
- net UART_RESET: no longer names the net of U1.28 (PD3)
- new net: Q1.1 (G), Q2.3 (C), R9.2
- new net: Q2.1 (B), R10.1
- new net GND1: J1.14 (GND), J1.20 (GND), J1.25 (GND), J1.30 (GND), J1.34 (GND), J1.39 (GND), J1.6 (GND), J1.9 (GND), J3.2 (Pin_2), J5.1 (Pin_1), Q1.2 (D)
- new net Vin: C3.1, J5.3 (Pin_3), R9.1, U2.3 (VI)
Other:
- note added: "3.3V Regulator\n"
- note added: "Power Switching Circuit\n\n\n"
- note removed: "Additional GPIO Output for Power Switching (if necessary)\n"
- moved on the sheet: C1, C2, D1, D2, D3, D4, D5, J2, R1, R2, R3, R4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

Commit message: New PCB
Parts:
- removed J3: Conn_01x04, Connector_PinHeader_2.54mm:PinHeader_1x04_P2.54mm_Horizontal, symbol Connector_Generic:Conn_01x04
- removed J4: Conn_01x03, FlightBridgePCB:EXTERNAL_TELEM, symbol Connector_Generic:Conn_01x03
- removed R7, R8: 0, Resistor_SMD:R_0805_2012Metric_Pad1.20x1.40mm_HandSolder, symbol Device:R
- removed U2: L78L33_TO92, Package_TO_SOT_THT:TO-92_Inline, symbol Regulator_Linear:L78L33_TO92
- added J3: Conn_01x03, Connector_PinHeader_2.54mm:PinHeader_1x03_P2.54mm_Horizontal, symbol Connector_Generic:Conn_01x03
- added J4: Conn_01x04, Connector_PinHeader_2.54mm:PinHeader_1x04_P2.54mm_Horizontal, symbol Connector_Generic:Conn_01x04
- added U2: MCP1700-3302E_TO92, Package_TO_SOT_THT:TO-92_Inline, symbol Regulator_Linear:MCP1700-3302E_TO92
Connections:
- net UART_SBUS is gone; now on net MOSI: J1.8 (GPIO14/TXD), U1.2 (PE0)
- net +3V3: now also J4.1 (Pin_1), U2.3 (VO)
- net +5V: now also J3.1 (Pin_1)
- net GND: now also J4.2 (Pin_2), U2.1 (GND)
- net GND1: now also J3.2 (Pin_2)
- net MISO: now also U1.3 (PE1); no longer U1.13 (PB3)
- net MOSI: now also J3.3 (Pin_3); no longer U1.12 (PB2)
- net UART_TELEM_PI: no longer U1.3 (PE1)
- net Vin: now also U2.2 (VI)
- net SDA: now reaches J1.3 (SDA/GPIO2)
- net SDA: now also J4.3 (Pin_3)
- net SCL: now reaches J1.5 (SCL/GPIO3)
- net SCL: now also J4.4 (Pin_4)
- net UART_TELEM: no longer names the net of U1.27 (PD2)
Other:
- note added: "Pi I2C breakout\n\n"
- note removed: "External Telemetry Input\n"
- note removed: "Telemetry Selector\n"
Changed lines of the file:
@@
 Wire Wire Line
 	5950 1100 5950 1150
-Text GLabel 6500 2550 2    50   BiDi ~ 0
+Text GLabel 5100 4050 0    50   BiDi ~ 0
 MOSI
-Text GLabel 6500 2650 2    50   BiDi ~ 0
+Text GLabel 5100 4250 0    50   BiDi ~ 0
 MISO
 Text GLabel 6500 2450 2    50   BiDi ~ 0
@@
 Text GLabel 1350 2600 0    50   Input ~ 0
 UART_TELEM_PI
-Text GLabel 5300 4150 0    50   Input ~ 0
+Text GLabel 5100 4150 0    50   Input ~ 0
 UART_SBUS
-Text GLabel 9550 1900 0    50   Input ~ 0
+Text GLabel 9550 1800 0    50   Input ~ 0
 UART_SBUS
-Text GLabel 9550 1800 0    50   Output ~ 0
-UART_TELEM_FC
-$Comp
-L Device:R R7
-U 1 1 606721A0
-P 9750 2700
-F 0 "R7" H 9820 2746 50  0000 L CNN
-F 1 "0" H 9820 2655 50  0000 L CNN
-F 2 "Resistor_SMD:R_0805_2012Metric_Pad1.20x1.40mm_HandSolder" V 9680 2700 50  0001 C CNN
-F 3 "~" H 9750 2700 50  0001 C CNN
-	1    9750 2700
-	1    0    0    -1
-$EndComp
-$Comp
-L Device:R R8
-U 1 1 60672D84
-P 9750 3000
-F 0 "R8" H 9820 3046 50  0000 L CNN
-F 1 "0" H 9820 2955 50  0000 L CNN
-F 2 "Resistor_SMD:R_0805_2012Metric_Pad1.20x1.40mm_HandSolder" V 9680 3000 50  0001 C CNN
-F 3 "~" H 9750 3000 50  0001 C CNN
-	1    9750 3000
-	1    0    0    -1
-$EndComp
-Text GLabel 9600 2850 0    50   Output ~ 0
-UART_TELEM
-Wire Wire Line
-	9600 2850 9750 2850
-Connection ~ 9750 2850
-Text Notes 9200 2350 0    50   ~ 0
-Telemetry Selector\n
-Text GLabel 10050 2550 2    50   Input ~ 0
-UART_TELEM_FC
-Wire Wire Line
-	9750 2550 10050 2550
-$Comp
-L Connector_Generic:Conn_01x03 J4
-U 1 1 6067E30D
-P 9550 3800
-F 0 "J4" H 9630 3842 50  0000 L CNN
-F 1 "Conn_01x03" H 9630 3751 50  0000 L CNN
-F 2 "FlightBridgePCB:EXTERNAL_TELEM" H 9550 3800 50  0001 C CNN
-F 3 "~" H 9550 3800 50  0001 C CNN
-	1    9550 3800
-	1    0    0    -1
-$EndComp
-Text Notes 9200 3400 0    50   ~ 0
-External Telemetry Input\n
-Text GLabel 9350 3900 0    50   Output ~ 0
-UART_TELEM_EXT
-$Comp
-L power:+5V #PWR0112
-U 1 1 6068215D
-P 9350 3700
-F 0 "#PWR0112" H 9350 3550 50  0001 C CNN
-F 1 "+5V" V 9365 3828 50  0000 L CNN
-F 2 "" H 9350 3700 50  0001 C CNN
-F 3 "" H 9350 3700 50  0001 C CNN
-	1    9350 3700
-	0    -1   -1   0
-$EndComp
-$Comp
-L power:GND #PWR0113
-U 1 1 60682A5F
-P 9350 3800
-F 0 "#PWR0113" H 9350 3550 50  0001 C CNN
-F 1 "GND" V 9355 3672 50  0000 R CNN
-F 2 "" H 9350 3800 50  0001 C CNN
-F 3 "" H 9350 3800 50  0001 C CNN
-	1    9350 3800
-	0    1    1    0
-$EndComp
-Text GLabel 10050 3150 2    50   Input ~ 0
-UART_TELEM_EXT
-Wire Wire Line
-	9750 3150 10050 3150
-Text GLabel 6500 4350 2    50   Input ~ 0
-UART_TELEM
-Text GLabel 5300 4250 0    50   Output ~ 0
-UART_TELEM_PI
 Text GLabel 1350 3600 0    50   Output ~ 0
 ABORT
@@
 ~POWER_EN~
 $Comp
-L Regulator_Linear:L78L33_TO92 U2
-U 1 1 607B052B
-P 2150 5500
-F 0 "U2" H 2150 5742 50  0000 C CNN
-F 1 "L78L33_TO92" H 2150 5651 50  0000 C CNN
-F 2 "Package_TO_SOT_THT:TO-92_Inline" H 2150 5725 50  0001 C CIN
-F 3 "http://www.st.com/content/ccc/resource/technical/document/datasheet/15/55/e5/aa/23/5b/43/fd/CD00000446.pdf/files/CD00000446.pdf/jcr:content/translations/en.CD00000446.pdf" H 2150 5450 50  0001 C CNN
-	1    2150 5500
-	1    0    0    -1
-$EndComp
-$Comp
 L Device:C C3
 U 1 1 607B28FC
@@
 	1400 7250 1350 7250
 $Comp
-L Connector_Generic:Conn_01x04 J3
-U 1 1 608B8E7D
-P 9750 1700
-F 0 "J3" H 9830 1692 50  0000 L CNN
-F 1 "Conn_01x04" H 9830 1601 50  0000 L CNN
-F 2 "Connector_PinHeader_2.54mm:PinHeader_1x04_P2.54mm_Horizontal" H 9750 1700 50  0001 C CNN
-F 3 "~" H 9750 1700 50  0001 C CNN
-	1    9750 1700
-	1    0    0    -1
-$EndComp
-$Comp
 L Connector:Raspberry_Pi_2_3 J1
 U 1 1 60669113
@@
 $EndComp
 Connection ~ 3150 1850
+Wire Wire Line
+	5300 4150 5200 4150
+Wire Wire Line
+	5100 4050 5200 4050
+Wire Wire Line
+	5200 4050 5200 4150
+Connection ~ 5200 4150
+Wire Wire Line
+	5200 4150 5100 4150
+Wire Wire Line
+	5100 4250 5300 4250
+$Comp
+L Regulator_Linear:MCP1700-3302E_TO92 U2
+U 1 1 609851B3
+P 2150 5500
+F 0 "U2" H 2150 5258 50  0000 C CNN
+F 1 "MCP1700-3302E_TO92" H 2150 5349 50  0000 C CNN
+F 2 "Package_TO_SOT_THT:TO-92_Inline" H 2150 5300 50  0001 C CIN
+F 3 "http://ww1.microchip.com/downloads/en/DeviceDoc/20001826D.pdf" H 2150 5500 50  0001 C CNN
+	1    2150 5500
+	1    0    0    1
+$EndComp
+$Comp
+L Connector_Generic:Conn_01x03 J3
+U 1 1 609C188B
+P 9750 1700
+F 0 "J3" H 9830 1742 50  0000 L CNN
+F 1 "Conn_01x03" H 9830 1651 50  0000 L CNN
+F 2 "Connector_PinHeader_2.54mm:PinHeader_1x03_P2.54mm_Horizontal" H 9750 1700 50  0001 C CNN
+F 3 "~" H 9750 1700 50  0001 C CNN
+	1    9750 1700
+	1    0    0    -1
+$EndComp
+Text GLabel 2950 2800 2    50   Output ~ 0
+SDA
+Text GLabel 2950 2900 2    50   Output ~ 0
+SCL
+Text Notes 9200 2300 0    50   ~ 0
+Pi I2C breakout\n\n
+$Comp
+L Connector_Generic:Conn_01x04 J4
+U 1 1 60A1AD24
+P 9750 2550
+F 0 "J4" H 9830 2542 50  0000 L CNN
+F 1 "Conn_01x04" H 9830 2451 50  0000 L CNN
+F 2 "Connector_PinHeader_2.54mm:PinHeader_1x04_P2.54mm_Horizontal" H 9750 2550 50  0001 C CNN
+F 3 "~" H 9750 2550 50  0001 C CNN
+	1    9750 2550
+	1    0    0    -1
+$EndComp
+$Comp
+L power:+3V3 #PWR0112
+U 1 1 60A1E0CF
+P 9550 2450
+F 0 "#PWR0112" H 9550 2300 50  0001 C CNN
+F 1 "+3V3" H 9565 2623 50  0000 C CNN
+F 2 "" H 9550 2450 50  0001 C CNN
+F 3 "" H 9550 2450 50  0001 C CNN
+	1    9550 2450
+	0    -1   -1   0
+$EndComp
+$Comp
+L power:GND #PWR0113
+U 1 1 60A26F57
+P 9350 2550
+F 0 "#PWR0113" H 9350 2300 50  0001 C CNN
+F 1 "GND" H 9355 2377 50  0000 C CNN
+F 2 "" H 9350 2550 50  0001 C CNN
+F 3 "" H 9350 2550 50  0001 C CNN
+	1    9350 2550
+	0    1    -1   0
+$EndComp
+Wire Wire Line
+	9550 2550 9350 2550
+Text GLabel 9550 2650 0    50   Input ~ 0
+SDA
+Text GLabel 9550 2750 0    50   Input ~ 0
+SCL
 $EndSCHEMATC
